File: MCU.kicad_sch (KiCad schematic)
At the start: 0 parts

Commit message: Added Example Peripherals🐐
Changed lines of the file:
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@@
+		)
+	)
+	(hierarchical_label "example_IO_2"
+		(shape input)
+		(at 182.88 97.79 0)
+		(fields_autoplaced yes)
+		(effects
+			(font
+				(size 1.27 1.27)
+			)
+			(justify left)
+		)
+	)
+	(hierarchical_label "example_IO_1"
+		(shape input)
+		(at 182.88 88.9 0)
+		(fields_autoplaced yes)
+		(effects
+			(font
+				(size 1.27 1.27)
+			)
+			(justify left)
 		)
 	)
