File: CubeFlightComputer.kicad_sch (KiCad schematic)
At the start: 0 parts

Commit message: title✍️
Other:
- note added: "This is the parent sheet for the Irishsat Cubestat flight Computer. Here, heirarchical blocks will be made for each individual IC or large subsystem. By breaking it down in this way, collaboration is simple. To contribute, follow the guide in the contributing section of our github: https://github.com/1112luke/CubeFlightComputer. (github repo location subject to change) Once we build out this shee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"
- note removed: "This is the parent sheet for the Irishsat Cubestat flight Computer. Here, Heirarchical blocks will be made for each individual IC or large subsystem. By breaking it down in this way, collaboration is simple. To contribute, follow the guide in the contributing section of our github: https://github.com/1112luke/CubeFlightComputer. (github repo location subject to change) Once we build out this shee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"
- title: (none) -> Cubesat Computer
Changed lines of the file:
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@@
 	(generator_version "8.0")
 	(paper "A4")
+	(title_block
+		(title "Cubesat Computer")
+	)
 	(wire
 		(pts
@@
 		)
 	)
-	(text "This is the parent sheet for the Irishsat Cubestat \nflight Computer. Here, Heirarchical blocks will be \nmade for each individual IC or large subsystem.\nBy breaking it down in this way, collaboration is simple.\nTo contribute, follow the guide in the contributing section\nof our github:\nhttps://github.com/1112luke/CubeFlightComputer.\n(github repo location subject to change)\n\nOnce we build out this sheet with the relevant peripherals,\ncontributing is as easy as taking a crack at implementing \nany one of them"
+	(text "This is the parent sheet for the Irishsat Cubestat \nflight Computer. Here, heirarchical blocks will be \nmade for each individual IC or large subsystem.\nBy breaking it down in this way, collaboration is simple.\nTo contribute, follow the guide in the contributing section\nof our github:\nhttps://github.com/1112luke/CubeFlightComputer.\n(github repo location subject to change)\n\nOnce we build out this sheet with the relevant peripherals,\ncontributing is as easy as taking a crack at implementing \nany one of them"
 		(exclude_from_sim no)
 		(at 101.854 70.358 0)

Commit message: Added Example Peripherals🐐
Other:
- added sheet GPS (GPS.kicad_sch)
- added sheet Pin_Header (Pin_Header.kicad_sch)
- sheet MCU ports: added example_IO_1, example_IO_2; removed none

Commit message: Text Change✍️
Other:
- note added: "This is the parent sheet for the Irishsat Cubesat flight Computer. Here, heirarchical blocks will be made for each individual IC or large subsystem. By breaking it down in this way, collaboration is simple. To contribute, follow the guide in the contributing section of our github: https://github.com/1112luke/CubeFlightComputer. (github repo location subject to change) Once we build out this sheet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"
- note removed: "This is the parent sheet for the Irishsat Cubestat flight Computer. Here, heirarchical blocks will be made for each individual IC or large subsystem. By breaking it down in this way, collaboration is simple. To contribute, follow the guide in the contributing section of our github: https://github.com/1112luke/CubeFlightComputer. (github repo location subject to change) Once we build out this shee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"
Changed lines of the file:
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@@
 		)
 	)
-	(text "This is the parent sheet for the Irishsat Cubestat \nflight Computer. Here, heirarchical blocks will be \nmade for each individual IC or large subsystem.\nBy breaking it down in this way, collaboration is simple.\nTo contribute, follow the guide in the contributing section\nof our github:\nhttps://github.com/1112luke/CubeFlightComputer.\n(github repo location subject to change)\n\nOnce we build out this sheet with the relevant peripherals,\ncontributing is as easy as taking a crack at implementing \nany one of them"
+	(text "This is the parent sheet for the Irishsat Cubesat \nflight Computer. Here, heirarchical blocks will be \nmade for each individual IC or large subsystem.\nBy breaking it down in this way, collaboration is simple.\nTo contribute, follow the guide in the contributing section\nof our github:\nhttps://github.com/1112luke/CubeFlightComputer.\n(github repo location subject to change)\n\nOnce we build out this sheet with the relevant peripherals,\ncontributing is as easy as taking a crack at implementing \nany one of them"
 		(exclude_from_sim no)
 		(at 48.26 34.29 0)
